Commit message: Changes to get the linear 3dof arm working on thorvald

File: description/d435/_d435.urdf.xacro (robot description, xacro)
@@ -46,5 +46,5 @@
         <geometry>
           <!-- <box size="${d435_cam_width} ${d435_cam_height} ${d435_cam_depth}"/> -->
-          <mesh filename="package://yeet/description/d435/d435.dae" />
+          <mesh filename="package://rasberry_perception/description/d435/d435.dae" />
           <!--<mesh filename="package://realsense2_description/meshes/d435/d435.dae" />-->
         </geometry>
