Commit message: Split repository into project components

File: grasberry_manipulation/description/linear_3dof_arm.urdf.xacro (robot description, xacro)
@@ -9,5 +9,5 @@
             <origin xyz="0 0 0" rpy="0 0 0"/>
             <geometry>
-                <mesh filename="package://rasberry_perception/description/meshes/gripper_example.dae"/>
+                <mesh filename="package://grasberry_manipulation/description/meshes/gripper_example.dae"/>
             </geometry>
             <material name="aluminum"/>

Commit message: Renamed folder from linear to arm_3dof since it will support multiple 3dof arms

File: grasberry_manipulation/description/linear_3dof_arm.urdf.xacro (robot description, xacro)
@@ -2,5 +2,5 @@
 <robot name="gripper" xmlns:xacro="http://ros.org/wiki/xacro">
     <!-- Base link for arm home -->
-    <link name="linear_3dof_arm_home"/>
+    <link name="linear_arm_3dof_home"/>
     <!-- Gripper Model -->
     <material name="aluminum"><color rgba="0.5 0.5 0.5 1"/></material>
@@ -14,7 +14,7 @@
         </visual>
     </link>
-    <joint name="linear_3dof_arm_home_link_joint" type="fixed">
+    <joint name="linear_arm_3dof_home_link_joint" type="fixed">
         <origin xyz="0 0 0" rpy="0 0 0"/>
-        <parent link="linear_3dof_arm_home"/>
+        <parent link="linear_arm_3dof_home"/>
         <child link="linear_3dof_gripper_link"/>
     </joint>
@@ -29,5 +29,5 @@
     <joint name="linear_3dof_2d_camera_home_link_joint" type="fixed">
         <origin xyz="-0.255 -0.115 -0.0675" rpy="0 ${15*DEG2RAD} ${90*DEG2RAD}"/>
-        <parent link="linear_3dof_arm_home"/>
+        <parent link="linear_arm_3dof_home"/>
         <child link="linear_3dof_2d_camera_link"/>
     </joint>
